Commit message: Add Astro robot configuration and assets
- Introduced new Astro robot configuration in `protomotions/robot_configs/astro.py`.
- Added asset files for Astro robot including USD and YAML configurations.
- Implemented asset hash and configuration files for USD conversion.
- Updated factory to include Astro robot configuration.
- Created unit tests for Astro robot configuration validation.
- Adjusted global alignment weight in Astro YAML configuration.
- Enhanced USD conversion script to handle multi-dot filenames for IsaacLab compatibility.

File: protomotions/data/assets/urdf/for_retargeting/astro_v1.urdf (robot description, URDF)
Before this commit: robot astro, 37 links, 36 joints
Joints:
- removed joint head_joint
- added joint head_yaw_joint: type revolute, parent torso_link, child head_link, origin xyz=0.0100000000000734 0 0.0349999999999515 rpy=0 0 0, axis 0.000 0.000 1.000, limit lower=-0.610 upper=0.610 effort=10.000 velocity=20.940
